Commit message: update arm description

File: models/azure_kinectDK/ur10_kinect.urdf (robot description, URDF)
Before this commit: robot ur10_v2.SLDASM, 3 links, 2 joints
Links:
- removed link amount_Link
- added link base
- added link base_link_inertia, mass 4.0; collision mesh filename=package://models/ur10/collision/base.stl; visual mesh filename=package://models/ur10/visual/base.dae
- added link flange
- added link forearm_link, mass 4.27; collision mesh filename=package://models/ur10/collision/forearm.stl; visual mesh filename=package://models/ur10/visual/forearm.dae
- added link mount_Link, mass 0.183514785358204; collision mesh filename=package://models/azure_kinectDK/meshes/mount_v2.STL; visual mesh filename=package://models/azure_kinectDK/meshes/mount_v2.STL
- added link shoulder_link, mass 7.1; collision mesh filename=package://models/ur10/collision/shoulder.stl; visual mesh filename=package://models/ur10/visual/shoulder.dae
- added link tool0
- added link upper_arm_link, mass 12.7; collision mesh filename=package://models/ur10/collision/upperarm.stl; visual mesh filename=package://models/ur10/visual/upperarm.dae
- added link wrist_1_link, mass 2.0; collision mesh filename=package://models/ur10/collision/wrist1.stl; visual mesh filename=package://models/ur10/visual/wrist1.dae
- added link wrist_2_link, mass 2.0; collision mesh filename=package://models/ur10/collision/wrist2.stl; visual mesh filename=package://models/ur10/visual/wrist2.dae
- added link wrist_3_link, mass 0.365; collision mesh filename=package://models/ur10/collision/wrist3.stl; visual mesh filename=package://models/ur10/visual/wrist3.dae
- link base_link: mass 18.7683162355854 -> None; geometry 
- link camera_Link: geometry collision mesh filename=package://models/azure_kinectDK/meshes/Azure Kinect DK.STL; visual mesh filename=package://models/azure_kinectDK/meshes/Azure Kinect DK.STL
Joints:
- removed joint joint1
- removed joint joint2
- added joint base_link-base_fixed_joint: type fixed, parent base_link, child base, origin xyz=0 0 0 rpy=0 0 3.141592653589793
- added joint base_link-base_link_inertia: type fixed, parent base_link, child base_link_inertia, origin xyz=0 0 0 rpy=0 0 3.141592653589793
- added joint camera_joint: type fixed, parent mount_Link, child camera_Link, origin xyz=0 0.0735 -0.021 rpy=0 0 -3.1416, axis 0 0 0
- added joint elbow_joint: type revolute, parent upper_arm_link, child forearm_link, origin xyz=-0.612 0 0 rpy=0 0 0, axis 0 0 1, limit lower=-3.141592653589793 upper=3.141592653589793 effort=150.0 velocity=3.141592653589793
- added joint flange-tool0: type fixed, parent flange, child tool0, origin xyz=0 0 0 rpy=1.5707963267948966 0 1.5707963267948966
- added joint mount_joint: type fixed, parent base_link, child mount_Link, origin xyz=0 0.25609 1.428 rpy=1.5708 0 -3.1416, axis 0 0 0
- added joint shoulder_lift_joint: type revolute, parent shoulder_link, child upper_arm_link, origin xyz=0 0 0 rpy=1.570796327 0 0, axis 0 0 1, limit lower=-6.283185307179586 upper=6.283185307179586 effort=330.0 velocity=2.0943951023931953
- added joint shoulder_pan_joint: type revolute, parent base_link_inertia, child shoulder_link, origin xyz=0 0 0.1273 rpy=0 0 0, axis 0 0 1, limit lower=-6.283185307179586 upper=6.283185307179586 effort=330.0 velocity=2.0943951023931953
- added joint wrist_1_joint: type revolute, parent forearm_link, child wrist_1_link, origin xyz=-0.5723 0 0.163941 rpy=0 0 0, axis 0 0 1, limit lower=-6.283185307179586 upper=6.283185307179586 effort=56.0 velocity=3.141592653589793
- added joint wrist_2_joint: type revolute, parent wrist_1_link, child wrist_2_link, origin xyz=0 -0.1157 -2.373046667922381e-11 rpy=1.570796327 0 0, axis 0 0 1, limit lower=-6.283185307179586 upper=6.283185307179586 effort=56.0 velocity=3.141592653589793
- added joint wrist_3-flange: type fixed, parent wrist_3_link, child flange, origin xyz=0 0 0 rpy=0 -1.5707963267948966 -1.5707963267948966
- added joint wrist_3_joint: type revolute, parent wrist_2_link, child wrist_3_link, origin xyz=0 0.0922 -1.891053610911353e-11 rpy=1.570796326589793 3.141592653589793 3.141592653589793, axis 0 0 1, limit lower=-6.283185307179586 upper=6.283185307179586 effort=56.0 velocity=3.141592653589793

File: models/ur10/ur10.urdf (robot description, URDF)
Before this commit: robot ur10_robot, 11 links, 10 joints
Links:
- link base_link_inertia: geometry collision mesh filename=package://mujoco_wrappers/models/ur10/assets/base.stl; visual mesh filename=package://mujoco_wrappers/models/ur10/assets/base.dae
- link forearm_link: geometry collision mesh filename=package://mujoco_wrappers/models/ur10/assets/forearm.stl; visual mesh filename=package://mujoco_wrappers/models/ur10/assets/forearm.dae
- link shoulder_link: geometry collision mesh filename=package://mujoco_wrappers/models/ur10/assets/shoulder.stl; visual mesh filename=package://mujoco_wrappers/models/ur10/assets/shoulder.dae
- link upper_arm_link: geometry collision mesh filename=package://mujoco_wrappers/models/ur10/assets/upperarm.stl; visual mesh filename=package://mujoco_wrappers/models/ur10/assets/upperarm.dae
- link wrist_1_link: geometry collision mesh filename=package://mujoco_wrappers/models/ur10/assets/wrist1.stl; visual mesh filename=package://mujoco_wrappers/models/ur10/assets/wrist1.dae
- link wrist_2_link: geometry collision mesh filename=package://mujoco_wrappers/models/ur10/assets/wrist2.stl; visual mesh filename=package://mujoco_wrappers/models/ur10/assets/wrist2.dae
- link wrist_3_link: geometry collision mesh filename=package://mujoco_wrappers/models/ur10/assets/wrist3.stl; visual mesh filename=package://mujoco_wrappers/models/ur10/assets/wrist3.dae
